File: upper_board/upper_board.kicad_pcb (KiCad board)
At the start: 2 copper layers, 96.5 x 96.5 mm, 38 parts, among them J1 Conn_01x04, J2 Conn_01x04, SW1 SW_Push, SW10 SW_Push, SW11 SW_Push, SW12 SW_Push, SW13 SW_Push, SW14 SW_Push, SW15 SW_Push, SW16 SW_Push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

Commit message: lower board component placement
Other:
- outline, holes or cut-outs redrawn
Changed lines of the file:
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@@
     )
   )
+  (gr_circle (center 152.807 76.65) (end 155.807 76.65) (layer "Edge.Cuts") (width 0.1) (fill none))
+  (gr_circle (center 133.757 57.6) (end 136.757 57.6) (layer "Edge.Cuts") (width 0.1) (fill none))
+  (gr_circle (center 171.8 114.75) (end 174.8 114.75) (layer "Edge.Cuts") (width 0.1) (fill none))
   (gr_arc (start 193.04 121.92) (mid 191.552102 125.512102) (end 187.96 127) (layer "Edge.Cuts") (width 0.2))
+  (gr_circle (center 114.707 114.75) (end 117.707 114.75) (layer "Edge.Cuts") (width 0.1) (fill none))
+  (gr_circle (center 114.707 95.7) (end 117.707 95.7) (layer "Edge.Cuts") (width 0.1) (fill none))
+  (gr_circle (center 114.707 76.65) (end 117.707 76.65) (layer "Edge.Cuts") (width 0.1) (fill none))
   (gr_arc (start 96.52 35.56) (mid 98.007898 31.967898) (end 101.6 30.48) (layer "Edge.Cuts") (width 0.2))
   (gr_arc (start 101.6 127) (mid 98.007898 125.512102) (end 96.52 121.92) (layer "Edge.Cuts") (width 0.2))
+  (gr_circle (center 114.707 57.6) (end 117.707 57.6) (layer "Edge.Cuts") (width 0.1) (fill none))
+  (gr_circle (center 171.857 95.7) (end 174.857 95.7) (layer "Edge.Cuts") (width 0.1) (fill none))
   (gr_line (start 187.96 30.48) (end 101.6 30.48) (layer "Edge.Cuts") (width 0.1))
+  (gr_circle (center 171.857 57.6) (end 174.857 57.6) (layer "Edge.Cuts") (width 0.1) (fill none))
   (gr_line (start 193.04 35.56) (end 193.04 121.92) (layer "Edge.Cuts") (width 0.1))
   (gr_arc (start 187.96 30.48) (mid 191.552102 31.967898) (end 193.04 35.56) (layer "Edge.Cuts") (width 0.1))
+  (gr_circle (center 152.807 95.7) (end 155.807 95.7) (layer "Edge.Cuts") (width 0.1) (fill none))
+  (gr_circle (center 133.757 114.75) (end 136.757 114.75) (layer "Edge.Cuts") (width 0.1) (fill none))
+  (gr_circle (center 133.757 95.7) (end 136.757 95.7) (layer "Edge.Cuts") (width 0.1) (fill none))
+  (gr_circle (center 152.807 114.75) (end 155.807 114.75) (layer "Edge.Cuts") (width 0.1) (fill none))
+  (gr_circle (center 152.807 57.6) (end 155.807 57.6) (layer "Edge.Cuts") (width 0.1) (fill none))
   (gr_line (start 96.52 35.56) (end 96.52 121.92) (layer "Edge.Cuts") (width 0.1))
   (gr_line (start 101.6 127) (end 187.96 127) (layer "Edge.Cuts") (width 0.1))
+  (gr_circle (center 133.757 76.65) (end 136.757 76.65) (layer "Edge.Cuts") (width 0.1) (fill none))
+  (gr_circle (center 171.857 76.65) (end 174.857 76.65) (layer "Edge.Cuts") (width 0.1) (fill none))
   (gr_text "Upper Deck" (at 101.6 76.2 90) (layer "F.Cu")
     (effects (font (size 2 2) (thickness 0.3)))
